File: kicad/ek_right_hand_35_buttons/ek_right_hand_35_buttons.kicad_pcb (KiCad board)
At the start: 2 copper layers, 129.5 x 99.1 mm, 42 parts, among them J1 Conn_01x06_Socket, U1 74HC165, U2 74HC165

Commit message: Righ hand 35 first PCB with very bad tracks
Parts:
- removed REF** (x4): MountingHole_2.2mm_M2, MountingHole:MountingHole_2.2mm_M2
- added C3: 100nF, Capacitor_THT:C_Rect_L7.0mm_W2.5mm_P5.00mm, F.Cu at (161.2, 71.3)
- added C4: 100nF, Capacitor_THT:C_Rect_L7.0mm_W2.5mm_P5.00mm, F.Cu at (211.6, 71.3)
- added C5: 100nF, Capacitor_THT:C_Rect_L7.0mm_W2.5mm_P5.00mm, F.Cu at (258.0, 71.3)
- added R17: 10k, Resistor_THT:R_Axial_DIN0207_L6.3mm_D2.5mm_P10.16mm_Horizontal, F.Cu at (140.5, 53.3)
- added R18: 10k, Resistor_THT:R_Axial_DIN0207_L6.3mm_D2.5mm_P10.16mm_Horizontal, F.Cu at (144.5, 53.3)
- added R19: 10k, Resistor_THT:R_Axial_DIN0207_L6.3mm_D2.5mm_P10.16mm_Horizontal, F.Cu at (148.5, 53.3)
- added R20: 10k, Resistor_THT:R_Axial_DIN0207_L6.3mm_D2.5mm_P10.16mm_Horizontal, F.Cu at (152.5, 53.3)
- added R21: 10k, Resistor_THT:R_Axial_DIN0207_L6.3mm_D2.5mm_P10.16mm_Horizontal, F.Cu at (174.9, 53.3)
- added R22: 10k, Resistor_THT:R_Axial_DIN0207_L6.3mm_D2.5mm_P10.16mm_Horizontal, F.Cu at (178.9, 53.3)
- added R23: 10k, Resistor_THT:R_Axial_DIN0207_L6.3mm_D2.5mm_P10.16mm_Horizontal, F.Cu at (182.9, 53.3)
- added R24: 10k, Resistor_THT:R_Axial_DIN0207_L6.3mm_D2.5mm_P10.16mm_Horizontal, F.Cu at (186.9, 53.3)
- added R25: 10k, Resistor_THT:R_Axial_DIN0207_L6.3mm_D2.5mm_P10.16mm_Horizontal, F.Cu at (190.9, 53.3)
- added R26: 10k, Resistor_THT:R_Axial_DIN0207_L6.3mm_D2.5mm_P10.16mm_Horizontal, F.Cu at (194.9, 53.3)
- added R27: 10k, Resistor_THT:R_Axial_DIN0207_L6.3mm_D2.5mm_P10.16mm_Horizontal, F.Cu at (198.9, 53.3)
- added R28: 10k, Resistor_THT:R_Axial_DIN0207_L6.3mm_D2.5mm_P10.16mm_Horizontal, F.Cu at (202.9, 53.3)
- added R29: 10k, Resistor_THT:R_Axial_DIN0207_L6.3mm_D2.5mm_P10.16mm_Horizontal, F.Cu at (225.3, 53.3)
- added R30: 10k, Resistor_THT:R_Axial_DIN0207_L6.3mm_D2.5mm_P10.16mm_Horizontal, F.Cu at (229.3, 53.3)
- added R31: 10k, Resistor_THT:R_Axial_DIN0207_L6.3mm_D2.5mm_P10.16mm_Horizontal, F.Cu at (233.3, 53.3)
- added R32: 10k, Resistor_THT:R_Axial_DIN0207_L6.3mm_D2.5mm_P10.16mm_Horizontal, F.Cu at (237.3, 53.3)
- added R33: 10k, Resistor_THT:R_Axial_DIN0207_L6.3mm_D2.5mm_P10.16mm_Horizontal, F.Cu at (241.3, 53.3)
- added R34: 10k, Resistor_THT:R_Axial_DIN0207_L6.3mm_D2.5mm_P10.16mm_Horizontal, F.Cu at (245.3, 53.3)
- added R35: 10k, Resistor_THT:R_Axial_DIN0207_L6.3mm_D2.5mm_P10.16mm_Horizontal, F.Cu at (249.3, 53.3)
- added SW17: ~, Button_Switch_Keyboard:SW_Cherry_MX_1.00u_PCB, F.Cu at (141.6, 117.9)
- added SW18: ~, Button_Switch_Keyboard:SW_Cherry_MX_1.00u_PCB, F.Cu at (151.1, 99.9)
- added SW19: ~, Button_Switch_Keyboard:SW_Cherry_MX_1.00u_PCB, F.Cu at (160.5, 81.9)
- added SW20: ~, Button_Switch_Keyboard:SW_Cherry_MX_1.00u_PCB, F.Cu at (160.5, 117.9)
- added SW21: ~, Button_Switch_Keyboard:SW_Cherry_MX_1.00u_PCB, F.Cu at (169.9, 99.9)
- added SW22: ~, Button_Switch_Keyboard:SW_Cherry_MX_1.00u_PCB, F.Cu at (179.4, 81.9)
- added SW23: ~, Button_Switch_Keyboard:SW_Cherry_MX_1.00u_PCB, F.Cu at (179.4, 117.9)
- added SW24: ~, Button_Switch_Keyboard:SW_Cherry_MX_1.00u_PCB, F.Cu at (188.8, 99.9)
- added SW25: ~, Button_Switch_Keyboard:SW_Cherry_MX_1.00u_PCB, F.Cu at (198.3, 81.9)
- added SW26: ~, Button_Switch_Keyboard:SW_Cherry_MX_1.00u_PCB, F.Cu at (198.3, 117.9)
- added SW27: ~, Button_Switch_Keyboard:SW_Cherry_MX_1.00u_PCB, F.Cu at (207.8, 99.9)
- added SW28: ~, Button_Switch_Keyboard:SW_Cherry_MX_1.00u_PCB, F.Cu at (217.2, 81.9)
- added SW29: ~, Button_Switch_Keyboard:SW_Cherry_MX_1.00u_PCB, F.Cu at (217.2, 117.9)
- added SW30: ~, Button_Switch_Keyboard:SW_Cherry_MX_1.00u_PCB, F.Cu at (226.7, 99.9)
- added SW31: ~, Button_Switch_Keyboard:SW_Cherry_MX_1.00u_PCB, F.Cu at (236.1, 81.9)
- added SW32: ~, Button_Switch_Keyboard:SW_Cherry_MX_1.00u_PCB, F.Cu at (236.1, 117.9)
- added SW33: ~, Button_Switch_Keyboard:SW_Cherry_MX_1.00u_PCB, F.Cu at (245.6, 99.9)
- added SW34: ~, Button_Switch_Keyboard:SW_Cherry_MX_1.00u_PCB, F.Cu at (255.0, 81.9)
- added SW35: ~, Button_Switch_Keyboard:SW_Cherry_MX_1.00u_PCB, F.Cu at (255.0, 117.9)
- added U3: 74HC165, Package_DIP:DIP-16_W7.62mm, F.Cu at (167.2, 67.3)
- added U4: 74HC165, Package_DIP:DIP-16_W7.62mm, F.Cu at (217.6, 67.3)
- added U5: 74HC165, Package_DIP:DIP-16_W7.62mm, F.Cu at (264.0, 67.3)
- J1: value Conn_01x06_Socket -> Conn_01x06
- moved ? 8.22 mm to (30.5, 106.7)
- moved R13 7.92 mm to (124.5, 53.3)
- moved R1 7.92 mm to (39.7, 53.3)
- moved R2 7.92 mm to (43.7, 53.3)
- moved R3 7.92 mm to (47.7, 53.3)
- moved R4 7.92 mm to (51.7, 53.3)
- moved J1 7.92 mm to (30.7, 65.9)
- moved C1 7.92 mm to (60.4, 71.3)
- moved C2 7.92 mm to (110.8, 71.3)
- moved R10 7.92 mm to (94.1, 53.3)
- moved R11 7.92 mm to (98.1, 53.3)
- moved R12 7.92 mm to (102.1, 53.3)
- moved R14 7.92 mm to (128.5, 53.3)
- moved R15 7.92 mm to (132.5, 53.3)
- moved R16 7.92 mm to (136.5, 53.3)
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Connections:
- net S1 renamed /Buttons 01-08/SERIAL_IN
- net SERIAL renamed /Buttons 01-08/SERIAL_OUT
- U2 pad 10: S2 -> /Buttons 09-16/SERIAL_IN
Routing:
- net VCC: track 397.3 -> 1056.7 mm
- net GND: track 160.1 -> 383.0 mm
- net CLK INH: track 113.2 -> 292.9 mm
- net CLK: track 106.7 -> 282.2 mm
- net SH/~{LD}: track 120.0 -> 294.2 mm
- net Net-(U3-D0): track 0.00 -> 80.7 mm
- net Net-(U4-D7): track 0.00 -> 79.0 mm
- net Net-(U4-D1): track 0.00 -> 77.6 mm
- net Net-(U3-D6): track 0.00 -> 74.9 mm
- net Net-(U3-D3): track 0.00 -> 67.1 mm
- net Net-(U5-D2): track 0.00 -> 66.7 mm
- net Net-(U4-D4): track 0.00 -> 66.0 mm
- net Net-(U3-D7): track 0.00 -> 60.6 mm
- net Net-(U5-D0): track 0.00 -> 57.0 mm
- net Net-(U3-D1): track 0.00 -> 56.9 mm
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Other:
- board size 129.5 x 99.1 mm -> 254 x 99.1 mm

Commit message: Right hand 35 first PCB with better tracks
Parts:
- moved ? 3.38 mm to (32.1, 103.7)
- moved C2 1.62 mm to (109.1, 71.3)
- moved C3 1.62 mm to (159.5, 71.3)
- moved C4 1.62 mm to (209.9, 71.3)
- moved C5 1.62 mm to (256.3, 71.3)
- moved C1 1.42 mm to (58.9, 71.3)
Routing:
- net GND: track 383.0 -> 0.17 mm
- net VCC: track 1056.7 -> 959.0 mm
- net SH/~{LD}: track 294.2 -> 352.5 mm
- net CLK INH: track 292.9 -> 341.3 mm
- net CLK: track 282.2 -> 293.8 mm
- net Net-(U3-D3): track 67.1 -> 75.8 mm
- net Net-(U2-D2): track 70.8 -> 78.8 mm
- net Net-(U3-D0): track 80.7 -> 88.5 mm
- net Net-(U1-D1): track 75.1 -> 82.7 mm
- net Net-(U3-D6): track 74.9 -> 81.1 mm
- net Net-(U1-D7): track 79.6 -> 85.8 mm
- net Net-(U4-D7): track 79.0 -> 85.1 mm
- net Net-(U5-D2): track 66.7 -> 72.1 mm
- net Net-(U4-D1): track 77.6 -> 82.9 mm
- net Net-(U2-D7): track 43.9 -> 47.9 mm
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- added copper zone on B.Cu, net GND
- added copper zone on F.Cu, net GND

Commit message: Right hand 35 first PCB with copper pour
Parts:
- moved J1 12.2 mm to (35.5, 54.7)
- moved ? 11.7 mm to (38.0, 93.6)
- moved SW21 11.1 mm to (171.3, 88.9)
- moved SW28 11.1 mm to (218.6, 70.9)
- moved SW29 11.1 mm to (218.6, 106.9)
- moved SW10 11.1 mm to (105.2, 70.9)
- moved SW11 11.1 mm to (105.2, 106.9)
- moved SW3 11.1 mm to (57.9, 88.9)
- moved SW9 11.1 mm to (95.7, 88.9)
- moved C5 11.1 mm to (257.7, 60.3)
- moved SW1 11.1 mm to (48.5, 70.9)
- moved SW12 11.1 mm to (114.6, 88.9)
- moved SW13 11.1 mm to (124.1, 70.9)
- moved SW14 11.1 mm to (124.1, 106.9)
- moved SW15 11.1 mm to (133.5, 88.9)
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Connections:
- J1 pad 2: CLK -> SH/~{LD}
- J1 pad 3: /Buttons 01-08/SERIAL_OUT -> CLK
- J1 pad 5: SH/~{LD} -> /Buttons 01-08/SERIAL_OUT
Routing:
- net CLK: track 293.8 -> 347.6 mm
- net VCC: track 959.0 -> 951.0 mm
- net SH/~{LD}: track 352.5 -> 346.7 mm
- net Net-(U1-D3): track 33.3 -> 36.6 mm
- net /Buttons 09-16/SERIAL_IN: track 55.3 -> 58.5 mm
- net /Buttons 17-24/SERIAL_IN: track 55.7 -> 58.5 mm
- net /Buttons 25-32/SERIAL_IN: track 51.2 -> 53.9 mm
- net Net-(U5-D2): track 72.1 -> 74.5 mm
- net Net-(U4-D3): track 34.4 -> 36.8 mm
- net /Buttons 01-08/SERIAL_IN: track 55.4 -> 57.7 mm
- net Net-(U2-D2): track 78.8 -> 80.0 mm
- net CLK INH: track 341.3 -> 340.1 mm
- net Net-(U3-D3): track 75.8 -> 76.8 mm
- net /Buttons 01-08/SERIAL_OUT: track 34.6 -> 35.3 mm
- net Net-(U1-D0): track 45.8 -> 46.4 mm
Other:
- board size 254 x 99.1 mm -> 243.4 x 107 mm

Commit message: Right hand 35 first PCB with vias, holes & labels
Parts:
- added M1: MountingHole_3.2mm_M3, MountingHole:MountingHole_3.2mm_M3, F.Cu at (27.1, 34.0)
- added M2: MountingHole_3.2mm_M3, MountingHole:MountingHole_3.2mm_M3, F.Cu at (267.1, 34.0)
- added M3: MountingHole_3.2mm_M3, MountingHole:MountingHole_3.2mm_M3, F.Cu at (27.1, 124.0)
- added M4: MountingHole_3.2mm_M3, MountingHole:MountingHole_3.2mm_M3, F.Cu at (267.1, 124.0)
- moved J1 16.0 mm to (34.7, 38.7), turned to 90 degrees
- moved R1 7.11 mm to (34.8, 45.6)
- moved R10 7.11 mm to (89.2, 45.6)
- moved R11 7.11 mm to (93.2, 45.6)
- moved R12 7.11 mm to (97.2, 45.6)
- moved R13 7.11 mm to (119.6, 45.6)
- moved R14 7.11 mm to (123.6, 45.6)
- moved R15 7.11 mm to (127.6, 45.6)
- moved R16 7.11 mm to (131.6, 45.6)
- moved R17 7.11 mm to (135.6, 45.6)
- moved R18 7.11 mm to (139.6, 45.6)
- moved R19 7.11 mm to (143.6, 45.6)
- moved R2 7.11 mm to (38.8, 45.6)
- moved R20 7.11 mm to (147.6, 45.6)
- moved R21 7.11 mm to (170.0, 45.6)
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Routing:
- net CLK: track 347.6 -> 313.6 mm
- net SH/~{LD}: track 346.7 -> 313.7 mm
- net /Buttons 01-08/SERIAL_OUT: track 35.3 -> 13.1 mm
- net VCC: track 951.0 -> 964.7 mm
- net CLK INH: track 340.1 -> 328.1 mm
- net Net-(U3-D0): track 88.5 -> 84.5 mm
- net Net-(U2-D0): track 63.4 -> 59.4 mm
- net Net-(U2-D7): track 47.9 -> 44.1 mm
- net Net-(U3-D7): track 63.0 -> 59.3 mm
- net Net-(U4-D7): track 85.1 -> 81.9 mm
- net Net-(U1-D7): track 85.8 -> 82.9 mm
- net Net-(U4-D0): track 45.8 -> 43.0 mm
- net Net-(U3-D3): track 76.8 -> 74.6 mm
- net Net-(U4-D3): track 36.8 -> 34.6 mm
- net Net-(U3-D4): track 48.7 -> 46.4 mm
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Other:
- board size 243.4 x 107 mm -> 250 x 100 mm
- board text added: "${TITLE1} ${TITLE2} Version : ${VERSION}"
- board text added: "CLK"
- board text added: "CLK INH"
- board text added: "GND"
- board text added: "SERIAL"
- board text added: "SH/~{LD}"
- board text added: "VCC"
