File: kicad/ek_right_hand_35_buttons/ek_right_hand_35_buttons.kicad_pcb (KiCad board)
At the start: 2 copper layers, 250 x 100 mm, 86 parts, among them J1 Conn_01x06, M1 MountingHole_3.2mm_M3, M2 MountingHole_3.2mm_M3, M3 MountingHole_3.2mm_M3, M4 MountingHole_3.2mm_M3, U1 74HC165, U2 74HC165, U3 74HC165, U4 74HC165, U5 74HC165

Commit message: Right hand 35 condensed positions
Parts:
- moved C5 7.00 mm to (244.4, 59.8)
- moved M2 7.00 mm to (260.1, 34.0)
- moved M4 7.00 mm to (260.1, 124.0)
- moved U5 7.00 mm to (252.1, 55.8)
- moved R35 6.75 mm to (237.6, 45.6)
- moved R34 6.45 mm to (233.9, 45.6)
- moved R33 6.15 mm to (230.2, 45.6)
- moved R32 5.85 mm to (226.5, 45.6)
- moved R31 5.55 mm to (222.8, 45.6)
- moved R30 5.25 mm to (219.1, 45.6)
- moved R28 5.05 mm to (192.9, 45.6)
- moved C4 5.00 mm to (200.0, 59.8)
- moved U4 5.00 mm to (207.7, 55.8)
- moved R29 4.95 mm to (215.4, 45.6)
- moved R27 4.75 mm to (189.2, 45.6)
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Routing:
- net CLK INH: track 328.1 -> 321.1 mm
- net VCC: track 964.7 -> 958.6 mm
- net SH/~{LD}: track 313.7 -> 307.7 mm
- net CLK: track 313.6 -> 308.2 mm
- net Net-(U5-D2): track 73.7 -> 79.1 mm
- net Net-(U4-D3): track 34.6 -> 39.5 mm
- net Net-(U4-D2): track 52.2 -> 55.6 mm
- net Net-(U4-D7): track 81.9 -> 85.3 mm
- net Net-(U5-D1): track 38.6 -> 41.3 mm
- net Net-(U4-D6): track 38.2 -> 40.5 mm
- net Net-(U5-D0): track 55.8 -> 58.0 mm
- net /Buttons 09-16/SERIAL_IN: track 58.5 -> 56.4 mm
- net /Buttons 25-32/SERIAL_IN: track 53.9 -> 51.9 mm
- net /Buttons 17-24/SERIAL_IN: track 58.5 -> 56.5 mm
- net /Buttons 01-08/SERIAL_IN: track 57.7 -> 55.7 mm
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Other:
- board size 250 x 100 mm -> 243 x 100 mm

Commit message: Right hand 35 better vias
Routing:
- net Net-(U1-D1): track 80.8 -> 78.3 mm
- net Net-(U2-D6): track 56.7 -> 54.3 mm
- net Net-(U4-D6): track 40.5 -> 38.2 mm
- net Net-(U2-D1): track 42.1 -> 39.9 mm
- net Net-(U3-D1): track 58.0 -> 55.8 mm
- net Net-(U2-D3): track 46.9 -> 49.1 mm
- net Net-(U4-D1): track 82.6 -> 80.5 mm
- net Net-(U1-D6): track 37.7 -> 35.6 mm
- net Net-(U2-D4): track 24.8 -> 26.8 mm
- net Net-(U3-D4): track 45.3 -> 47.3 mm
- net Net-(U1-D4): track 66.2 -> 68.1 mm
- net Net-(U3-D6): track 79.8 -> 77.9 mm
- net Net-(U3-D3): track 75.6 -> 77.5 mm
- net Net-(U4-D3): track 39.5 -> 41.4 mm
- net Net-(U1-D3): track 34.1 -> 35.8 mm
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
Commit message: Right hand 35 vias and gerber
Routing:
- net Net-(U5-D1): track 40.4 -> 44.6 mm
- net SH/~{LD}: track 307.7 -> 310.7 mm
- net Net-(U2-D3): track 49.1 -> 51.5 mm
- net Net-(U3-D3): track 77.5 -> 79.8 mm
- net CLK INH: track 321.1 -> 323.0 mm
- net Net-(U2-D1): track 39.9 -> 39.3 mm
- net GND: vias 48 -> 152

Commit message: Right hand 35 vias and gerber
Routing:
- net /Buttons 17-24/SERIAL_IN: track 56.5 -> 57.2 mm
- net GND: vias 152 -> 196
