File: kicad/ek_right_hand_35_buttons/ek_right_hand_35_buttons.kicad_sch (KiCad schematic)
At the start: 1 part, among them J1 Conn_01x06

Commit message: Righ hand 35 first PCB with very bad tracks
Parts:
- J1: footprint (none) -> Connector_PinHeader_2.54mm:PinHeader_1x06_P2.54mm_Vertical
Changed lines of the file:
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@@
       (effects (font (size 1.27 1.27)) (justify left))
     )
-    (property "Footprint" "" (at 63.5 30.48 0)
+    (property "Footprint" "Connector_PinHeader_2.54mm:PinHeader_1x06_P2.54mm_Vertical" (at 63.5 30.48 0)
       (effects (font (size 1.27 1.27)) hide)
     )

Commit message: Right hand 35 first PCB with copper pour
Connections:
- net Buttons 01-08/SERIAL_OUT: now also J1.5 (Pin_5); no longer J1.3 (Pin_3)
- net CLK: now also J1.3 (Pin_3); no longer J1.2 (Pin_2)
- net SH/~{LD}: now also J1.2 (Pin_2); no longer J1.5 (Pin_5)
Changed lines of the file:
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@@
+    (stroke (width 0) (type default))
+  )
+  (wire (pts (xy 44.45 30.48) (xy 58.42 30.48))
     (stroke (width 0) (type default))
   )
@@
     (stroke (width 0) (type default))
   )
-  (wire (pts (xy 48.26 33.02) (xy 58.42 33.02))
+  (wire (pts (xy 25.4 35.56) (xy 58.42 35.56))
+    (stroke (width 0) (type default))
+  )
+  (wire (pts (xy 55.88 33.02) (xy 58.42 33.02))
+    (stroke (width 0) (type default))
+  )
+  (wire (pts (xy 55.88 27.94) (xy 58.42 27.94))
     (stroke (width 0) (type default))
   )
@@
     (stroke (width 0) (type default))
   )
-  (wire (pts (xy 36.83 35.56) (xy 58.42 35.56))
+  (wire (pts (xy 25.4 35.56) (xy 25.4 63.5))
     (stroke (width 0) (type default))
   )
@@
     (stroke (width 0) (type default))
   )
-  (wire (pts (xy 25.4 30.48) (xy 25.4 63.5))
-    (stroke (width 0) (type default))
-  )
-  (wire (pts (xy 44.45 27.94) (xy 58.42 27.94))
-    (stroke (width 0) (type default))
-  )
   (wire (pts (xy 27.94 67.31) (xy 27.94 63.5))
-    (stroke (width 0) (type default))
-  )
-  (wire (pts (xy 25.4 30.48) (xy 58.42 30.48))
     (stroke (width 0) (type default))
   )
@@
     (effects (font (size 1.27 1.27)) (justify left top))
   )
-  (global_label "SH{slash}~{LD}" (shape output) (at 36.83 35.56 180) (fields_autoplaced)
+  (global_label "SH{slash}~{LD}" (shape output) (at 55.88 27.94 180) (fields_autoplaced)
     (effects (font (size 1.27 1.27)) (justify right))
-    (property "Intersheetrefs" "${INTERSHEET_REFS}" (at 27.6762 35.56 0)
+    (property "Intersheetrefs" "${INTERSHEET_REFS}" (at 46.7262 27.94 0)
       (effects (font (size 1.27 1.27)) (justify right) hide)
     )
   )
-  (global_label "CLK" (shape output) (at 44.45 27.94 180) (fields_autoplaced)
+  (global_label "CLK" (shape output) (at 44.45 30.48 180) (fields_autoplaced)
     (effects (font (size 1.27 1.27)) (justify right))
-    (property "Intersheetrefs" "${INTERSHEET_REFS}" (at 37.8967 27.94 0)
+    (property "Intersheetrefs" "${INTERSHEET_REFS}" (at 37.8967 30.48 0)
       (effects (font (size 1.27 1.27)) (justify right) hide)
     )
   )
-  (global_label "CLK INH" (shape output) (at 48.26 33.02 180) (fields_autoplaced)
+  (global_label "CLK INH" (shape output) (at 55.88 33.02 180) (fields_autoplaced)
     (effects (font (size 1.27 1.27)) (justify right))
-    (property "Intersheetrefs" "${INTERSHEET_REFS}" (at 37.4733 33.02 0)
+    (property "Intersheetrefs" "${INTERSHEET_REFS}" (at 45.0933 33.02 0)
       (effects (font (size 1.27 1.27)) (justify right) hide)
     )

Commit message: Right hand 35 first PCB with vias, holes & labels
Other:
- title: ${TITLE} -> ${TITLE1}  - ${TITLE2}
Changed lines of the file:
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@@
   (paper "A4")
   (title_block
-    (title "${TITLE}")
+    (title "${TITLE1}  - ${TITLE2}")
     (date "2023-08-15")
     (rev "${VERSION}")
